Commit message: Add functioning livox HAP sensor.

File: vl400_description/urdf/sentry.xacro (robot description, xacro)
@@ -105,7 +105,15 @@
     </gazebo>
     <!-- Velodyne VLP-16 (gz-sim gpu_lidar / lidar sensor) -->
-    <xacro:include filename="$(find vl400_description)/urdf/velodyne_vlp16.urdf.xacro"/>
+    <!-- <xacro:include filename="$(find vl400_description)/urdf/velodyne_vlp16.urdf.xacro"/>
         <xacro:VLP-16 parent="sentry_link" name="velodyne" topic="/velodyne_points" organize_cloud="${organize_cloud}" hz="10" samples="440" gpu="${gpu}">
         <origin xyz="0.47 0.42 0.41" rpy="-1.5707 0 0" />
-    </xacro:VLP-16>
+    </xacro:VLP-16> -->
+    <!-- Livox HAP (gz-sim gpu_lidar + livox_laser_simulation plugin,
+         see urdf/livox_hap.xacro). Publishes the resampled Livox
+         cloud on /livox/lidar/pointcloud2 in frame livox_hap_frame,
+         with TF world -> livox_hap_frame. -->
+    <xacro:include filename="$(find vl400_description)/urdf/livox_hap.xacro"/>
+    <xacro:livox_hap parent="sentry_link" name="livox_hap" topic="/livox_hap" ros_topic="/livox/lidar/pointcloud2" frame_id="livox_hap_frame">
+      <origin xyz="0.47 0.30 0.41" rpy="-1.5707 0 0"/>
+    </xacro:livox_hap>
 </robot>

File: vl400_description/urdf/vl400.xacro (robot description, xacro)
@@ -454,5 +454,8 @@
 </joint>
 <!-- ======================= gz-sim systems ======================= -->
-  <!-- Publish wheel joint states (bridged to ROS /joint_states) -->
+  <!-- Publish wheel joint states (bridged to ROS /joint_states).
+       The lidar mount joint is listed too so robot_state_publisher
+       publishes the livox_hap_link transform (the lidar cloud itself
+       is anchored on the world frame by the livox plugin). -->
   <gazebo>
     <plugin filename="gz-sim-joint-state-publisher-system" name="gz::sim::systems::JointStatePublisher">
@@ -461,4 +464,5 @@
       <joint_name>right_wheel_fake_joint</joint_name>
       <joint_name>left_wheel_fake_joint</joint_name>
+      <joint_name>livox_hap_joint</joint_name>
     </plugin>
   </gazebo>
