Commit message: Fix tf tree

File: vl400_description/urdf/livox_hap.xacro (robot description, xacro)
@@ -13,5 +13,5 @@
          (scan_patterns/HAP.csv, installed to share/vl400_description)
          and publishes a Livox-style PointCloud2 on <ros_topic> plus
-         the TF  world -> <frame_id>.
+         the TF  sentry_link -> <frame_id>.
        * The plugin library liblivox_laser_simulation.so is built by
          this package (see CMakeLists.txt) and found through
@@ -39,7 +39,7 @@
             topic:=/livox_hap
             ros_topic:=/livox/lidar/pointcloud2
-            frame_id:=livox_hap_frame
+            frame_id:=livox_hap_link
             csv:=HAP.csv
-            hz:=1
+            hz:=10
             h_samples:=611
             v_samples:=141
@@ -139,5 +139,5 @@
           <ros_topic>${ros_topic}</ros_topic>
           <frame_name>${frame_id}</frame_name>
-          <parent_frame_id>world</parent_frame_id>
+          <parent_frame_id>sentry_link</parent_frame_id>
           <use_inf>false</use_inf>
         </plugin>

File: vl400_description/urdf/sentry.xacro (robot description, xacro)
@@ -4,5 +4,5 @@
     <xacro:arg name="organize_cloud" default="false"/>
     <xacro:property name="organize_cloud" value="$(arg organize_cloud)" />
-    <!-- #######################################################################################################-->
+    <!-- ######### SENTRY link ######### -->
     <link name="sentry_link">
       <visual>
@@ -24,9 +24,13 @@
     <joint name="sentry_joint" type="fixed">
      <origin rpy="1.5707 0 0" xyz="${-wheel_radius-0.5} 0.4 ${base_z_size/2}"/>
-      <child link="sentry_link" />
-      <parent link="chassis_link"/>
+     <parent link="chassis_link"/>
+     <child link="sentry_link"/>
     </joint>
+    <gazebo reference="sentry_link">
+      <mu1>0.05</mu1>
+      <mu2>0.05</mu2>
+    </gazebo>
     <!--#########   DURO LINK (IMU) #########-->
-      <link name="duro_link">
+      <link name="imu_link">
         <inertial>
           <mass value="0.01"/>
@@ -47,16 +51,12 @@
         <origin xyz="0.27 0.40 0.41" rpy="-1.5707 0 0"/>
         <parent link="sentry_link"/>
-        <child link="duro_link"/>
+        <child link="imu_link"/>
       </joint>
-      <gazebo reference="sentry_link">
-        <mu1>0.05</mu1>
-        <mu2>0.05</mu2>
-      </gazebo>
-      <gazebo reference="duro_link">
+      <gazebo reference="imu_link">
         <sensor name="imu_sensor" type="imu">
           <always_on>true</always_on>
           <update_rate>100</update_rate>
           <topic>/imu</topic>
-          <gz_frame_id>duro_link</gz_frame_id>
+          <gz_frame_id>imu_link</gz_frame_id>
           <imu/>
         </sensor>
@@ -65,8 +65,7 @@
           <update_rate>10</update_rate>
           <topic>/mag</topic>
-          <gz_frame_id>duro_link</gz_frame_id>
+          <gz_frame_id>imu_link</gz_frame_id>
         </sensor>
       </gazebo>
-    <!--#########  END DURO LINK #########-->
     <!--######### GPS SENSOR #########-->
       <link name="gps_link">
@@ -88,5 +87,5 @@
       <joint name="joint_gps" type="fixed">
         <origin xyz="0 0 0.055" rpy="0 0 0"/>
-        <parent link="duro_link"/>
+        <parent link="sentry_link"/>
         <child link="gps_link"/>
       </joint>
@@ -99,5 +98,20 @@
         </sensor>
       </gazebo>
-    <!--######### END GPS SENSOR #########-->
+    <!-- gz-sim's Sensors system only CREATES the non-rendering sensors
+         above (imu, magnetometer, navsat); their data is published by
+         dedicated systems. Without these three plugins the gz topics
+         /imu, /mag and /fix receive no messages and the ROS bridge
+         forwards nothing. They are model-level plugins so they work
+         in every world the robot is spawned into. -->
+    <gazebo>
+      <plugin filename="gz-sim-imu-system" name="gz::sim::systems::Imu"/>
+    </gazebo>
+    <gazebo>
+      <plugin filename="gz-sim-magnetometer-system" name="gz::sim::systems::Magnetometer"/>
+    </gazebo>
+    <gazebo>
+      <plugin filename="gz-sim-navsat-system" name="gz::sim::systems::NavSat"/>
+    </gazebo>
+    <!--######### LiDAR Sensors (Velodyni, livox HAP) #########-->
     <gazebo reference="velodyne_base_link">
         <mu1>0.05</mu1>

File: vl400_description/urdf/vl400.xacro (robot description, xacro)
@@ -62,9 +62,9 @@
    </collision>
 </link>
-<link name="base_footprint" />
+<link name="base_link" />
 <joint name="chassis_joint" type="fixed">
   <origin xyz="0 0 ${-(base_z_size/2 + wheel_vertical_offset)}" rpy="0 0 0" />
-  <parent link="chassis_link" />
-  <child link="base_footprint" />
+  <parent link="base_link" />
+  <child link="chassis_link" />
 </joint>
 <!-- #######################################################################################################-->
