Commit message: remove description pkg and move to parent directory vl400_sim

File: urdf/livox_hap.xacro (robot description, xacro)
@@ -11,5 +11,5 @@
        * The livox_laser_simulation plugin attached to the sensor
          resamples that depth image onto the measured HAP scan pattern
-         (scan_patterns/HAP.csv, installed to share/vl400_description)
+         (scan_patterns/HAP.csv, installed to share/vl400_sim)
          and publishes a Livox-style PointCloud2 on <ros_topic> plus
          the TF  sentry_link -> <frame_id>.
@@ -124,5 +124,5 @@
                          2 = PointCloud2 xyz+intensity+tag+line+timestamp
                              (Livox PointXYZRTLT, the default),
-                         3 = vl400_description/msg/CustomMsg.
+                         3 = vl400_sim/msg/CustomMsg.
              samples x hz = point_rate = output points per second. -->
         <plugin filename="liblivox_laser_simulation.so"

File: urdf/sentry.xacro (robot description, xacro)
@@ -4,10 +4,10 @@
     <xacro:arg name="organize_cloud" default="false"/>
     <xacro:property name="organize_cloud" value="$(arg organize_cloud)" />
-    <!-- #######################################################################################################-->
+    <!-- ######### SENTRY link ######### -->
     <link name="sentry_link">
       <visual>
           <origin rpy="0 0 0" xyz="0 0 0"/>
           <geometry>
-             <mesh filename="package://vl400_description/meshes/Sentry.STL" scale="0.0012 0.0012 0.0012"/>
+             <mesh filename="package://vl400_sim/meshes/Sentry.STL" scale="0.0012 0.0012 0.0012"/>
           </geometry>
           <material name="silver">
@@ -18,5 +18,5 @@
         <origin rpy="0 0 0" xyz="0 0 0"/>
         <geometry>
-              <mesh filename="package://vl400_description/meshes/Sentry.STL" scale="0.0012 0.0012 0.0012"/>
+              <mesh filename="package://vl400_sim/meshes/Sentry.STL" scale="0.0012 0.0012 0.0012"/>
           </geometry>
       </collision>
@@ -24,9 +24,13 @@
     <joint name="sentry_joint" type="fixed">
      <origin rpy="1.5707 0 0" xyz="${-wheel_radius-0.5} 0.4 ${base_z_size/2}"/>
-      <child link="sentry_link" />
-      <parent link="chassis_link"/>
+     <parent link="chassis_link"/>
+     <child link="sentry_link"/>
     </joint>
+    <gazebo reference="sentry_link">
+      <mu1>0.05</mu1>
+      <mu2>0.05</mu2>
+    </gazebo>
     <!--#########   DURO LINK (IMU) #########-->
-      <link name="duro_link">
+      <link name="imu_link">
         <inertial>
           <mass value="0.01"/>
@@ -47,16 +51,12 @@
         <origin xyz="0.27 0.40 0.41" rpy="-1.5707 0 0"/>
         <parent link="sentry_link"/>
-        <child link="duro_link"/>
+        <child link="imu_link"/>
       </joint>
-      <gazebo reference="sentry_link">
-        <mu1>0.05</mu1>
-        <mu2>0.05</mu2>
-      </gazebo>
-      <gazebo reference="duro_link">
+      <gazebo reference="imu_link">
         <sensor name="imu_sensor" type="imu">
           <always_on>true</always_on>
           <update_rate>100</update_rate>
           <topic>/imu</topic>
-          <gz_frame_id>duro_link</gz_frame_id>
+          <gz_frame_id>imu_link</gz_frame_id>
           <imu/>
         </sensor>
@@ -65,8 +65,7 @@
           <update_rate>10</update_rate>
           <topic>/mag</topic>
-          <gz_frame_id>duro_link</gz_frame_id>
+          <gz_frame_id>imu_link</gz_frame_id>
         </sensor>
       </gazebo>
-    <!--#########  END DURO LINK #########-->
     <!--######### GPS SENSOR #########-->
       <link name="gps_link">
@@ -88,5 +87,5 @@
       <joint name="joint_gps" type="fixed">
         <origin xyz="0 0 0.055" rpy="0 0 0"/>
-        <parent link="duro_link"/>
+        <parent link="sentry_link"/>
         <child link="gps_link"/>
       </joint>
@@ -99,5 +98,20 @@
         </sensor>
       </gazebo>
-    <!--######### END GPS SENSOR #########-->
+    <!-- gz-sim's Sensors system only CREATES the non-rendering sensors
+         above (imu, magnetometer, navsat); their data is published by
+         dedicated systems. Without these three plugins the gz topics
+         /imu, /mag and /fix receive no messages and the ROS bridge
+         forwards nothing. They are model-level plugins so they work
+         in every world the robot is spawned into. -->
+    <gazebo>
+      <plugin filename="gz-sim-imu-system" name="gz::sim::systems::Imu"/>
+    </gazebo>
+    <gazebo>
+      <plugin filename="gz-sim-magnetometer-system" name="gz::sim::systems::Magnetometer"/>
+    </gazebo>
+    <gazebo>
+      <plugin filename="gz-sim-navsat-system" name="gz::sim::systems::NavSat"/>
+    </gazebo>
+    <!--######### LiDAR Sensors (Velodyni, livox HAP) #########-->
     <gazebo reference="velodyne_base_link">
         <mu1>0.05</mu1>
@@ -105,7 +119,15 @@
     </gazebo>
     <!-- Velodyne VLP-16 (gz-sim gpu_lidar / lidar sensor) -->
-    <xacro:include filename="$(find vl400_description)/urdf/velodyne_vlp16.urdf.xacro"/>
+    <!-- <xacro:include filename="$(find vl400_sim)/urdf/velodyne_vlp16.urdf.xacro"/>
         <xacro:VLP-16 parent="sentry_link" name="velodyne" topic="/velodyne_points" organize_cloud="${organize_cloud}" hz="10" samples="440" gpu="${gpu}">
         <origin xyz="0.47 0.42 0.41" rpy="-1.5707 0 0" />
-    </xacro:VLP-16>
+    </xacro:VLP-16> -->
+    <!-- Livox HAP (gz-sim gpu_lidar + livox_laser_simulation plugin,
+         see urdf/livox_hap.xacro). Publishes the resampled Livox
+         cloud on /livox/lidar/pointcloud2 in frame livox_hap_frame,
+         with TF world -> livox_hap_frame. -->
+    <xacro:include filename="$(find vl400_sim)/urdf/livox_hap.xacro"/>
+    <xacro:livox_hap parent="sentry_link" name="livox_hap" topic="/livox_hap" ros_topic="/livox/lidar/pointcloud2" frame_id="livox_hap_frame">
+      <origin xyz="0.47 0.30 0.41" rpy="-1.5707 0 0"/>
+    </xacro:livox_hap>
 </robot>

File: urdf/velodyne_vlp16.urdf.xacro (robot description, xacro)
@@ -24,10 +24,10 @@
       <visual>
         <geometry>
-          <mesh filename="package://vl400_description/meshes/VLP16_base_1.dae" />
+          <mesh filename="package://vl400_sim/meshes/VLP16_base_1.dae" />
         </geometry>
       </visual>
       <visual>
         <geometry>
-          <mesh filename="package://vl400_description/meshes/VLP16_base_2.dae" />
+          <mesh filename="package://vl400_sim/meshes/VLP16_base_2.dae" />
         </geometry>
       </visual>
@@ -53,5 +53,5 @@
         <origin xyz="0 0 -0.0377" />
         <geometry>
-          <mesh filename="package://vl400_description/meshes/VLP16_scan.dae" />
+          <mesh filename="package://vl400_sim/meshes/VLP16_scan.dae" />
         </geometry>
       </visual>

File: urdf/vl400.xacro (robot description, xacro)
@@ -13,5 +13,5 @@
   <xacro:property name="wheel_radius" value="0.45" />
   <!-- ADD SENTRY and sensors xacro -->
-  <xacro:include filename="$(find vl400_description)/urdf/sentry.xacro"/>
+  <xacro:include filename="$(find vl400_sim)/urdf/sentry.xacro"/>
   <!--  INERTIA COMPUTATION-->
     <!--cylinder-->
@@ -90,5 +90,5 @@
     <origin rpy="0 0 -1.5707" xyz="0 0 0"/>
     <geometry>
-      <mesh filename="package://vl400_description/meshes/wheel_v2.stl" scale="0.0013 0.0015 0.0015"/>
+      <mesh filename="package://vl400_sim/meshes/wheel_v2.stl" scale="0.0013 0.0015 0.0015"/>
     </geometry>
     <material name="black">
@@ -125,5 +125,5 @@
     <origin rpy="0 0 1.5707" xyz="0 0 0"/>
     <geometry>
-      <mesh filename="package://vl400_description/meshes/wheel_v2.stl" scale="0.0013 0.0015 0.0015"/>
+      <mesh filename="package://vl400_sim/meshes/wheel_v2.stl" scale="0.0013 0.0015 0.0015"/>
     </geometry>
     <material name="black">
@@ -198,5 +198,5 @@
     <origin rpy="0 0 0" xyz="0 ${y_off} 0"/>
     <geometry>
-      <mesh filename="package://vl400_description/meshes/belt_band.dae"/>
+      <mesh filename="package://vl400_sim/meshes/belt_band.dae"/>
     </geometry>
     <material name="tread">
@@ -387,5 +387,5 @@
       <origin rpy="0 0 0" xyz="0 0 0"/>
       <geometry>
-         <mesh filename="package://vl400_description/meshes/Hood.STL" scale="0.002 0.0015 0.0015"/>
+         <mesh filename="package://vl400_sim/meshes/Hood.STL" scale="0.002 0.0015 0.0015"/>
       </geometry>
       <material name="green">
@@ -404,5 +404,5 @@
       <origin rpy="0 0 0" xyz="0 0 0"/>
       <geometry>
-         <mesh filename="package://vl400_description/meshes/Tubular.STL" scale="0.0023 0.001 0.003"/>
+         <mesh filename="package://vl400_sim/meshes/Tubular.STL" scale="0.0023 0.001 0.003"/>
       </geometry>
       <material name="orange">
@@ -421,5 +421,5 @@
       <origin rpy="0 0 0" xyz="0 0 0"/>
       <geometry>
-         <mesh filename="package://vl400_description/meshes/Mulcher_v2.STL" scale="0.0012 0.0012 0.0012"/>
+         <mesh filename="package://vl400_sim/meshes/Mulcher_v2.STL" scale="0.0012 0.0012 0.0012"/>
       </geometry>
       <material name="green">
@@ -430,5 +430,5 @@
     <origin rpy="0 0 0" xyz="0 0 0"/>
     <geometry>
-        <mesh filename="package://vl400_description/meshes/Mulcher_v2.STL" scale="0.0012 0.0012 0.0012"/>
+        <mesh filename="package://vl400_sim/meshes/Mulcher_v2.STL" scale="0.0012 0.0012 0.0012"/>
       </geometry>
   </collision>

Commit message: Improve livox HAP pattern and speedup livox frequency by decreasing some resolution

File: urdf/livox_hap.xacro (robot description, xacro)
@@ -4,9 +4,10 @@
        Livox HAP lidar for gz-sim, mounted on the sentry.
        How it works:
-       * The gpu_lidar sensor renders a dense depth image. Its LaserScan
-         on <topic> doubles as a width x height distance image (this is
-         what the plugin resamples), and it also publishes a raw
-         PointCloudPacked on <topic>/points (bridged to the ROS topic
-         /livox_hap_points in config/bridge.yaml).
+       * The gpu_lidar sensor renders a coarse depth image (a range
+         lookup table). Its LaserScan on <topic> doubles as a
+         width x height distance image (this is what the plugin
+         resamples at the exact CSV pattern directions), and it also
+         publishes a raw PointCloudPacked on <topic>/points (bridged
+         to the ROS topic /livox_hap_points in config/bridge.yaml).
        * The livox_laser_simulation plugin attached to the sensor
          resamples that depth image onto the measured HAP scan pattern
@@ -33,7 +34,11 @@
        HAP field of view is 120 x 25 deg (scan pattern azimuth
        -60.25..60.25 deg, elevation -13.25..13.25 deg). The depth
-       image covers +/-61 x +/-14 deg at 0.2 deg/pixel, which fully
-       covers the scan pattern (the plugin checks this and refuses to
-       publish otherwise).
+       image covers +/-61 x +/-14 deg at 0.5 deg/pixel (245 x 57 =
+       ~14k rays instead of 86k), which fully covers the scan pattern
+       (the plugin checks this and refuses to publish otherwise) and
+       keeps the sensor render cheap. The CSV holds one full
+       non-repetitive pattern: 1048576 points at 2.2 us/point
+       (~453k points/s), so samples x hz reproduces the real HAP rate
+       (45300 x 10 Hz).
        ================================================================== -->
   <xacro:property name="M_PI" value="3.1415926535897931"/>
@@ -46,6 +51,6 @@
             csv:=HAP.csv
             hz:=10
-            h_samples:=611
-            v_samples:=141
+            h_samples:=245
+            v_samples:=57
             min_angle:=-${61.0*M_PI/180.0}
             max_angle:=${61.0*M_PI/180.0}
@@ -54,8 +59,8 @@
             min_range:=0.1
             max_range:=200.0
-            samples:=20000
+            samples:=45300
             downsample:=1
             line_count:=4
-            point_rate:=200000
+            point_rate:=453000
             cloud_type:=2">
     <link name="${name}_link">
@@ -123,5 +128,7 @@
         </lidar>
         <!-- Resamples the depth image above onto the HAP scan pattern
-             and publishes the ROS PointCloud2 (no TF). The plugin must sit
+             and publishes the ROS PointCloud2 (no TF). Points keep the
+             exact CSV pattern directions; the depth image supplies only
+             the range. The plugin must sit
              inside the <sensor>: it attaches to the sensor entity.
              cloud_type: 1 = PointCloud2 xyz,

File: urdf/sentry.xacro (robot description, xacro)
@@ -15,9 +15,13 @@
           </material>
         </visual>
+      <!-- Box proxy matching the mesh AABB (0.55 x 0.64 x 0.60 m).
+           Mesh collisions on the robot trigger the ODE trimesh-trimesh
+           path against the terrain mesh (grind + crash); see the note
+           on tool_link in vl400.xacro. -->
       <collision>
-        <origin rpy="0 0 0" xyz="0 0 0"/>
+        <origin rpy="0 0 0" xyz="0.272 0.318 0.411"/>
         <geometry>
-              <mesh filename="package://vl400_sim/meshes/Sentry.STL" scale="0.0012 0.0012 0.0012"/>
-          </geometry>
+          <box size="0.545 0.637 0.599"/>
+        </geometry>
       </collision>
     </link>

File: urdf/vl400.xacro (robot description, xacro)
@@ -436,9 +436,14 @@
       </material>
     </visual>
-  <collision>
-    <origin rpy="0 0 0" xyz="0 0 0"/>
-    <geometry>
-        <mesh filename="package://vl400_sim/meshes/Mulcher_v2.STL" scale="0.0012 0.0012 0.0012"/>
-      </geometry>
+  <!-- Box proxy matching the mesh AABB (1.98 x 0.53 x 1.27 m). A mesh
+       collision on the robot makes ODE take the trimesh-trimesh path
+       against the terrain mesh: constant contact grinds the sim to a
+       halt and eventually crashes it. Primitive proxies keep the fast
+       collision path. -->
+  <collision>
+    <origin rpy="0 0 0" xyz="0.99 0.265 0.634"/>
+    <geometry>
+      <box size="1.98 0.53 1.27"/>
+    </geometry>
   </collision>
 </link>
