Commit message: Fix vl400 model in rviz2, there was a problem in the tf_tree that is being used by the robot_state_publisher

File: urdf/sentry.xacro (robot description, xacro)
@@ -59,5 +59,16 @@
           <topic>/imu</topic>
           <gz_frame_id>imu_link</gz_frame_id>
-          <imu/>
+          <imu>
+            <angular_velocity>
+              <x><noise type="gaussian"><mean>0.0</mean><stddev>2e-4</stddev></noise></x>
+              <y><noise type="gaussian"><mean>0.0</mean><stddev>2e-4</stddev></noise></y>
+              <z><noise type="gaussian"><mean>0.0</mean><stddev>2e-4</stddev></noise></z>
+            </angular_velocity>
+            <linear_acceleration>
+              <x><noise type="gaussian"><mean>0.0</mean><stddev>1.7e-2</stddev></noise></x>
+              <y><noise type="gaussian"><mean>0.0</mean><stddev>1.7e-2</stddev></noise></y>
+              <z><noise type="gaussian"><mean>0.0</mean><stddev>1.7e-2</stddev></noise></z>
+            </linear_acceleration>
+          </imu>
         </sensor>
         <sensor name="mag_sensor" type="magnetometer">
@@ -67,4 +78,10 @@
           <gz_frame_id>imu_link</gz_frame_id>
         </sensor>
+      </gazebo>
+      <gazebo>
+        <plugin filename="gz-sim-imu-system" name="gz::sim::systems::Imu"/>
+      </gazebo>
+      <gazebo>
+        <plugin filename="gz-sim-magnetometer-system" name="gz::sim::systems::Magnetometer"/>
       </gazebo>
     <!--######### GPS SENSOR #########-->
@@ -87,30 +104,18 @@
       <joint name="joint_gps" type="fixed">
         <origin xyz="0 0 0.055" rpy="0 0 0"/>
-        <parent link="sentry_link"/>
+        <parent link="imu_link"/>
         <child link="gps_link"/>
       </joint>
-      <gazebo reference="gps_link">
-        <sensor name="gps_sensor" type="navsat">
-          <always_on>true</always_on>
-          <update_rate>10</update_rate>
-          <topic>/fix</topic>
-          <gz_frame_id>gps_link</gz_frame_id>
-        </sensor>
-      </gazebo>
-    <!-- gz-sim's Sensors system only CREATES the non-rendering sensors
-         above (imu, magnetometer, navsat); their data is published by
-         dedicated systems. Without these three plugins the gz topics
-         /imu, /mag and /fix receive no messages and the ROS bridge
-         forwards nothing. They are model-level plugins so they work
-         in every world the robot is spawned into. -->
-    <gazebo>
-      <plugin filename="gz-sim-imu-system" name="gz::sim::systems::Imu"/>
-    </gazebo>
-    <gazebo>
-      <plugin filename="gz-sim-magnetometer-system" name="gz::sim::systems::Magnetometer"/>
-    </gazebo>
-    <gazebo>
-      <plugin filename="gz-sim-navsat-system" name="gz::sim::systems::NavSat"/>
-    </gazebo>
+        <gazebo reference="gps_link">
+            <sensor name="gps_sensor" type="navsat">
+                <always_on>true</always_on>
+                <update_rate>10</update_rate>
+                <topic>/fix</topic>
+                <gz_frame_id>gps_link</gz_frame_id>
+            </sensor>
+        </gazebo>
+        <gazebo>
+            <plugin filename="gz-sim-navsat-system" name="gz::sim::systems::NavSat"/>
+        </gazebo>
     <!--######### LiDAR Sensors (Velodyni, livox HAP) #########-->
     <gazebo reference="velodyne_base_link">
@@ -118,13 +123,10 @@
         <mu2>0.05</mu2>
     </gazebo>
-    <!-- Velodyne VLP-16 (gz-sim gpu_lidar / lidar sensor) -->
+    <!-- Velodyne VLP-16 -->
     <!-- <xacro:include filename="$(find vl400_sim)/urdf/velodyne_vlp16.urdf.xacro"/>
         <xacro:VLP-16 parent="sentry_link" name="velodyne" topic="/velodyne_points" organize_cloud="${organize_cloud}" hz="10" samples="440" gpu="${gpu}">
         <origin xyz="0.47 0.42 0.41" rpy="-1.5707 0 0" />
     </xacro:VLP-16> -->
-    <!-- Livox HAP (gz-sim gpu_lidar + livox_laser_simulation plugin,
-         see urdf/livox_hap.xacro). Publishes the resampled Livox
-         cloud on /livox/lidar/pointcloud2 in frame livox_hap_frame,
-         with TF world -> livox_hap_frame. -->
+    <!-- Livox HAP -->
     <xacro:include filename="$(find vl400_sim)/urdf/livox_hap.xacro"/>
     <xacro:livox_hap parent="sentry_link" name="livox_hap" topic="/livox_hap" ros_topic="/livox/lidar/pointcloud2" frame_id="livox_hap_frame">

File: urdf/vl400.xacro (robot description, xacro)
@@ -380,4 +380,13 @@
   </xacro:if>
 </xacro:macro>
+<!-- Emit <joint_name> elements for one track's plate joints. Used in the
+     JointStatePublisher whitelist below so the tread plates get TF. -->
+<xacro:macro name="track_joint_names" params="prefix n">
+  <xacro:if value="${n > 0}">
+    <joint_name>${prefix}_arm_j_${n - 1}</joint_name>
+    <joint_name>${prefix}_slide_j_${n - 1}</joint_name>
+    <xacro:track_joint_names prefix="${prefix}" n="${n - 1}"/>
+  </xacro:if>
+</xacro:macro>
 <xacro:track_plates side="left" y_off="0.13" prefix="track_anim_left" n="${track_anim_plate_count}"/>
 <xacro:track_plates side="right" y_off="0.15" prefix="track_anim_right" n="${track_anim_plate_count}"/>
@@ -457,5 +466,11 @@
        The lidar mount joint is listed too so robot_state_publisher
        publishes the livox_hap_link transform (the lidar cloud itself
-       is anchored on the world frame by the livox plugin). -->
+       is anchored on the world frame by the livox plugin).
+       The track assembly joints and all tread plate joints are listed
+       as well: robot_state_publisher only publishes TF for joints it
+       receives states for, so without these the track links and plates
+       have no transform and RViz cannot display them. The plate states
+       are the live TrackVisual animation, so RViz shows the treads
+       circulating around the loop. -->
   <gazebo>
     <plugin filename="gz-sim-joint-state-publisher-system" name="gz::sim::systems::JointStatePublisher">
@@ -465,4 +480,8 @@
       <joint_name>left_wheel_fake_joint</joint_name>
       <joint_name>livox_hap_joint</joint_name>
+      <joint_name>track_left_wheel_joint</joint_name>
+      <joint_name>track_right_wheel_joint</joint_name>
+      <xacro:track_joint_names prefix="track_anim_left" n="${track_anim_plate_count}"/>
+      <xacro:track_joint_names prefix="track_anim_right" n="${track_anim_plate_count}"/>
     </plugin>
   </gazebo>

Commit message: Add Zed 2i camera with depth. Fix some frames issue

File: urdf/sentry.xacro (robot description, xacro)
@@ -6,4 +6,11 @@
     <!-- ######### SENTRY link ######### -->
     <link name="sentry_link">
+      <!-- Sensor mast, ~3 kg; CoM at the mesh AABB center, inertia of
+           the 0.545 x 0.637 x 0.599 m box. -->
+      <inertial>
+        <origin xyz="0.272 0.318 0.411"/>
+        <mass value="3"/>
+        <inertia ixx="0.191" ixy="0" ixz="0" iyy="0.164" iyz="0" izz="0.176"/>
+      </inertial>
       <visual>
           <origin rpy="0 0 0" xyz="0 0 0"/>
@@ -32,6 +39,6 @@
     </joint>
     <gazebo reference="sentry_link">
-      <mu1>0.05</mu1>
-      <mu2>0.05</mu2>
+      <mu1>0.3</mu1>
+      <mu2>0.3</mu2>
     </gazebo>
     <!--#########   DURO LINK (IMU) #########-->
@@ -65,7 +72,7 @@
           <imu>
             <angular_velocity>
-              <x><noise type="gaussian"><mean>0.0</mean><stddev>2e-4</stddev></noise></x>
-              <y><noise type="gaussian"><mean>0.0</mean><stddev>2e-4</stddev></noise></y>
-              <z><noise type="gaussian"><mean>0.0</mean><stddev>2e-4</stddev></noise></z>
+              <x><noise type="gaussian"><mean>0.0</mean><stddev>2e-3</stddev></noise></x>
+              <y><noise type="gaussian"><mean>0.0</mean><stddev>2e-3</stddev></noise></y>
+              <z><noise type="gaussian"><mean>0.0</mean><stddev>2e-3</stddev></noise></z>
             </angular_velocity>
             <linear_acceleration>
@@ -135,5 +142,7 @@
     <xacro:include filename="$(find vl400_sim)/urdf/livox_hap.xacro"/>
     <xacro:livox_hap parent="sentry_link" name="livox_hap" topic="/livox_hap" ros_topic="/livox/lidar/pointcloud2" frame_id="livox_hap_link">
-      <origin xyz="0.47 0.30 0.41" rpy="-1.5707 0 0"/>
+      <origin xyz="0.45 0.33 0.41" rpy="-1.5707 0 0"/>
     </xacro:livox_hap>
+    <!-- Zed 2i Camera -->
+    <xacro:include filename="$(find vl400_sim)/urdf/zed2i_camera.xacro"/>
 </robot>

File: urdf/vl400.xacro (robot description, xacro)
@@ -45,5 +45,9 @@
   </xacro:macro>
   <link name="chassis_link">
-   <xacro:box_inertial  x="${base_x_size}" y="${base_y_size}" z="${base_z_size}" mass="50" />
+   <!-- 1200 kg hull: ~333 kg/m^3 of bounding volume, in the band for a
+        compact tracked machine (real CTLs/tractors run 200-400). With
+        tracks, wheels, mulcher and panels the robot totals ~2.4 t,
+        giving ~21 kPa ground pressure on the two belt footprints. -->
+   <xacro:box_inertial  x="${base_x_size}" y="${base_y_size}" z="${base_z_size}" mass="1200" />
    <visual>
     <origin xyz="0 0 0" rpy="0 0 0" />
@@ -70,5 +74,5 @@
 <!-- #######################################################################################################-->
 <link name="right_wheel_link">
-   <xacro:cylinder_inertia  r="${wheel_radius}" l="${wheel_length}"  mass="7" />
+   <xacro:cylinder_inertia  r="${wheel_radius}" l="${wheel_length}"  mass="60" />
   <collision>
   <origin rpy="0 1.5707 1.5707" xyz="0 0 0"/>
@@ -86,5 +90,5 @@
 <!-- #######################################################################################################-->
 <link name="right_wheel_fake_link">
-   <xacro:cylinder_inertia  r="${wheel_radius}" l="${wheel_length}"  mass="0.1" />
+   <xacro:cylinder_inertia  r="${wheel_radius}" l="${wheel_length}"  mass="60" />
    <visual>
     <origin rpy="0 0 -1.5707" xyz="0 0 0"/>
@@ -105,5 +109,5 @@
 <!-- #######################################################################################################-->
 <link name="left_wheel_link">
-   <xacro:cylinder_inertia  r="${wheel_radius}" l="${wheel_length}"  mass="7" />
+   <xacro:cylinder_inertia  r="${wheel_radius}" l="${wheel_length}"  mass="60" />
   <collision>
   <origin rpy="0 1.5707 1.5707" xyz="0 0 0"/>
@@ -121,5 +125,5 @@
 <!-- #######################################################################################################-->
 <link name="left_wheel_fake_link">
-   <xacro:cylinder_inertia  r="${wheel_radius}" l="${wheel_length}"  mass="0.1" />
+   <xacro:cylinder_inertia  r="${wheel_radius}" l="${wheel_length}"  mass="60" />
    <visual>
     <origin rpy="0 0 1.5707" xyz="0 0 0"/>
@@ -140,4 +144,6 @@
 <!-- #######################################################################################################-->
 <link name="support_right_wheel_link">
+  <!-- Support roller, ~5 kg (0.4 m dia x 0.3 m rubber roller). -->
+  <xacro:cylinder_inertia r="0.2" l="${wheel_length}" mass="5"/>
   <visual>
       <origin rpy="0 1.5707 1.5707" xyz="0 0 0"/>
@@ -163,4 +169,6 @@
 <!-- #######################################################################################################-->
 <link name="support_left_wheel_link">
+  <!-- Support roller, ~5 kg (0.4 m dia x 0.3 m rubber roller). -->
+  <xacro:cylinder_inertia r="0.2" l="${wheel_length}" mass="5"/>
   <visual>
       <origin rpy="0 1.5707 1.5707" xyz="0 0 0"/>
@@ -227,48 +235,53 @@
 </xacro:macro>
 <gazebo reference="track_left_wheel_link">
-  <mu1>0.7</mu1>
-  <mu2>150</mu2>
+  <!-- Rubber track on soil: ~1.0 longitudinal grip, ~0.6 lateral so
+       the machine skid-steers. fdir1 is lateral (y), so mu1 applies
+       laterally and mu2 longitudinally. -->
+  <mu1>0.6</mu1>
+  <mu2>1.0</mu2>
   <fdir1>0 1 0</fdir1>
 </gazebo>
 <gazebo reference="track_right_wheel_link">
-  <mu1>0.7</mu1>
-  <mu2>150</mu2>
+  <mu1>0.6</mu1>
+  <mu2>1.0</mu2>
   <fdir1>0 1 0</fdir1>
 </gazebo>
-<!-- Skid plates: on rough terrain the chassis belly, the tail stabilizer
-     and the support wheels can rest on bumps while the belt hangs in
-     the air. Near-zero friction lets those parts slide instead of
-     anchoring the robot; the belt supplies all the traction. Note the
+<!-- Non-driving contact surfaces. The hull has ~21 cm ground clearance
+     and the belt is the lowest point, so these only touch on large
+     bumps or side slopes; they get realistic material friction
+     (steel hull/stabilizer/mulcher ~0.3 on soil, rubber rollers and
+     road wheels ~0.8) while the belt supplies the traction. Note the
      URDF->SDF converter applies each block to the collisions of that
      exact link only, so every fixed-jointed body part needs its own
      block (they get lumped into chassis_link but keep their names). -->
 <gazebo reference="chassis_link">
-  <mu1>0.05</mu1>
-  <mu2>0.05</mu2>
+  <mu1>0.3</mu1>
+  <mu2>0.3</mu2>
 </gazebo>
 <gazebo reference="stabilizer_link">
-  <mu1>0.05</mu1>
-  <mu2>0.05</mu2>
+  <mu1>0.3</mu1>
+  <mu2>0.3</mu2>
 </gazebo>
 <gazebo reference="support_left_wheel_link">
-  <mu1>0.05</mu1>
-  <mu2>0.05</mu2>
+  <mu1>0.8</mu1>
+  <mu2>0.8</mu2>
 </gazebo>
 <gazebo reference="support_right_wheel_link">
-  <mu1>0.05</mu1>
-  <mu2>0.05</mu2>
+  <mu1>0.8</mu1>
+  <mu2>0.8</mu2>
 </gazebo>
 <gazebo reference="tool_link">
-  <mu1>0.05</mu1>
-  <mu2>0.05</mu2>
-</gazebo>
-<!-- Wheels inside the belt: spin freely if they ever touch the ground. -->
+  <mu1>0.3</mu1>
+  <mu2>0.3</mu2>
+</gazebo>
+<!-- Road wheels inside the belt: rubber, they sit ~9 mm above the
+     belt bottom and only touch on soft ground. -->
 <gazebo reference="right_wheel_link">
-  <mu1>0.05</mu1>
-  <mu2>0.05</mu2>
+  <mu1>0.8</mu1>
+  <mu2>0.8</mu2>
 </gazebo>
 <gazebo reference="left_wheel_link">
-  <mu1>0.05</mu1>
-  <mu2>0.05</mu2>
+  <mu1>0.8</mu1>
+  <mu2>0.8</mu2>
 </gazebo>
 <!-- Tracked-vehicle conversion: the track links carry the belt        -->
@@ -287,6 +300,9 @@
            robot backwards onto its tail stabilizer). -->
       <origin xyz="1.38 0 0.3755"/>
-      <mass value="5"/>
-      <inertia ixx="0.37" ixy="0" ixz="0" iyy="0.55" iyz="0" izz="0.5"/>
+      <!-- 250 kg per side: rubber belt + steel grousers + rollers of a
+           ~1.9 m track. Inertia of a 2.0 x 0.3 x 0.9 m box about its
+           center. -->
+      <mass value="250"/>
+      <inertia ixx="18.75" ixy="0" ixz="0" iyy="100.21" iyz="0" izz="85.21"/>
     </inertial>
   <xacro:belt_collisions y_off="0.13"/>
@@ -307,6 +323,9 @@
            robot backwards onto its tail stabilizer). -->
       <origin xyz="1.38 0 0.3755"/>
-      <mass value="5"/>
-      <inertia ixx="0.37" ixy="0" ixz="0" iyy="0.55" iyz="0" izz="0.5"/>
+      <!-- 250 kg per side: rubber belt + steel grousers + rollers of a
+           ~1.9 m track. Inertia of a 2.0 x 0.3 x 0.9 m box about its
+           center. -->
+      <mass value="250"/>
+      <inertia ixx="18.75" ixy="0" ixz="0" iyy="100.21" iyz="0" izz="85.21"/>
     </inertial>
   <xacro:belt_collisions y_off="0.15"/>
@@ -333,7 +352,7 @@
   <link name="${prefix}_arm_${i}">
     <inertial>
-      <mass value="0.01"/>
+      <mass value="0.5"/>
       <origin xyz="0 0 0"/>
-      <inertia ixx="1e-6" ixy="0" ixz="0" iyy="1e-6" iyz="0" izz="1e-6"/>
+      <inertia ixx="5e-4" ixy="0" ixz="0" iyy="5e-4" iyz="0" izz="5e-4"/>
     </inertial>
   </link>
@@ -347,7 +366,9 @@
   <link name="${prefix}_plate_${i}">
     <inertial>
-      <mass value="0.01"/>
+      <!-- Steel grouser, ~1 kg; inertia of the 0.016 x 0.30 x 0.06
+           cleat box about its center. -->
+      <mass value="1.0"/>
       <origin xyz="0 0 0"/>
-      <inertia ixx="1e-6" ixy="0" ixz="0" iyy="1e-6" iyz="0" izz="1e-6"/>
+      <inertia ixx="0.0078" ixy="0" ixz="0" iyy="0.00032" iyz="0" izz="0.0075"/>
     </inertial>
     <!-- One cleat riding the continuous band. Link frame: x radial
@@ -393,4 +414,11 @@
 <!-- #######################################################################################################-->
 <link name="stetic_body_link">
+  <!-- Hood panel, ~40 kg; CoM at the mesh AABB center, inertia of the
+       1.42 x 0.71 x 1.68 m box. -->
+  <inertial>
+    <origin xyz="0.717 0.354 0.849"/>
+    <mass value="40"/>
+    <inertia ixx="11.06" ixy="0" ixz="0" iyy="16.14" iyz="0" izz="8.42"/>
+  </inertial>
   <visual>
       <origin rpy="0 0 0" xyz="0 0 0"/>
@@ -410,4 +438,11 @@
 <!-- #######################################################################################################-->
 <link name="stetic_tube_link">
+  <!-- Tubular frame, ~25 kg; CoM at the mesh AABB center, inertia of
+       the 1.64 x 0.80 x 1.30 m box. -->
+  <inertial>
+    <origin xyz="0.822 0.470 0.653"/>
+    <mass value="25"/>
+    <inertia ixx="4.89" ixy="0" ixz="0" iyy="9.13" iyz="0" izz="6.93"/>
+  </inertial>
   <visual>
       <origin rpy="0 0 0" xyz="0 0 0"/>
@@ -427,4 +462,11 @@
 <!-- #######################################################################################################-->
 <link name="tool_link">
+  <!-- Mulcher head, ~400 kg (2 m wide drum + housing); CoM at the mesh
+       AABB center, inertia of the 1.98 x 0.53 x 1.27 m box. -->
+  <inertial>
+    <origin xyz="0.99 0.265 0.634"/>
+    <mass value="400"/>
+    <inertia ixx="63.13" ixy="0" ixz="0" iyy="184.44" iyz="0" izz="140.04"/>
+  </inertial>
   <visual>
       <origin rpy="0 0 0" xyz="0 0 0"/>
@@ -455,4 +497,6 @@
 <!-- #######################################################################################################-->
 <link name="stabilizer_link">
+  <!-- Tail stabilizer, ~5 kg. -->
+  <xacro:box_inertial x="0.2" y="0.2" z="0.2" mass="5"/>
   <collision>
     <origin rpy="0 0 0" xyz="0 0 0"/>
