Commit message: Fix imu and gps tf on the SENTRY. Improve the robot friction to be more realistic

File: urdf/sentry.xacro (robot description, xacro)
@@ -60,5 +60,5 @@
       </link>
       <joint name="joint_imu" type="fixed">
-        <origin xyz="0.27 0.40 0.41" rpy="-1.5707 0 0"/>
+        <origin xyz="0.27 0.30 0.41" rpy="-1.5707 0 0"/>
         <parent link="sentry_link"/>
         <child link="imu_link"/>
@@ -114,6 +114,6 @@
       </link>
       <joint name="joint_gps" type="fixed">
-        <origin xyz="0 0 0.055" rpy="0 0 0"/>
-        <parent link="imu_link"/>
+        <origin xyz="0.27 0.45 0.41" rpy="-1.59 0 0"/>
+        <parent link="sentry_link"/>
         <child link="gps_link"/>
       </joint>

File: urdf/vl400.xacro (robot description, xacro)
@@ -45,9 +45,18 @@
   </xacro:macro>
   <link name="chassis_link">
-   <!-- 1200 kg hull: ~333 kg/m^3 of bounding volume, in the band for a
-        compact tracked machine (real CTLs/tractors run 200-400). With
-        tracks, wheels, mulcher and panels the robot totals ~2.4 t,
-        giving ~21 kPa ground pressure on the two belt footprints. -->
-   <xacro:box_inertial  x="${base_x_size}" y="${base_y_size}" z="${base_z_size}" mass="1200" />
+   <!-- ~700 kg hull lump: frame + panels + engine + hydraulic
+        equipment. The mass center sits in the lower third of the hull
+        box (drivetrain and hydraulic oil are low; hood and cab are
+        sheet steel). The real machine climbs ~60 deg slopes, which
+        requires a low mass center; the hull is the biggest lever for
+        it. Inertia: box about the shifted center (parallel axis
+        adds mass*d^2 to ixx/iyy). -->
+   <inertial>
+     <mass value="700"/>
+     <origin xyz="0 0 -0.3"/>
+     <inertia ixx="${0.0833333 * 700 * (base_y_size*base_y_size + base_z_size*base_z_size) + 700 * 0.09}" ixy="0" ixz="0"
+              iyy="${0.0833333 * 700 * (base_x_size*base_x_size + base_z_size*base_z_size) + 700 * 0.09}" iyz="0"
+              izz="${0.0833333 * 700 * (base_x_size*base_x_size + base_y_size*base_y_size)}"/>
+   </inertial>
    <visual>
     <origin xyz="0 0 0" rpy="0 0 0" />
@@ -74,5 +83,6 @@
 <!-- #######################################################################################################-->
 <link name="right_wheel_link">
-   <xacro:cylinder_inertia  r="${wheel_radius}" l="${wheel_length}"  mass="60" />
+   <!-- Road wheel: rubber-tyred steel wheel, ~150 kg. -->
+   <xacro:cylinder_inertia  r="${wheel_radius}" l="${wheel_length}"  mass="150" />
   <collision>
   <origin rpy="0 1.5707 1.5707" xyz="0 0 0"/>
@@ -90,5 +100,7 @@
 <!-- #######################################################################################################-->
 <link name="right_wheel_fake_link">
-   <xacro:cylinder_inertia  r="${wheel_radius}" l="${wheel_length}"  mass="60" />
+   <!-- Visual-only rear wheel copy (spin animation via DiffDrive):
+        minimum link mass, it is not real hardware. -->
+   <xacro:cylinder_inertia  r="${wheel_radius}" l="${wheel_length}"  mass="5" />
    <visual>
     <origin rpy="0 0 -1.5707" xyz="0 0 0"/>
@@ -109,5 +121,6 @@
 <!-- #######################################################################################################-->
 <link name="left_wheel_link">
-   <xacro:cylinder_inertia  r="${wheel_radius}" l="${wheel_length}"  mass="60" />
+   <!-- Road wheel: rubber-tyred steel wheel, ~150 kg. -->
+   <xacro:cylinder_inertia  r="${wheel_radius}" l="${wheel_length}"  mass="150" />
   <collision>
   <origin rpy="0 1.5707 1.5707" xyz="0 0 0"/>
@@ -125,5 +138,7 @@
 <!-- #######################################################################################################-->
 <link name="left_wheel_fake_link">
-   <xacro:cylinder_inertia  r="${wheel_radius}" l="${wheel_length}"  mass="60" />
+   <!-- Visual-only rear wheel copy (spin animation via DiffDrive):
+        minimum link mass, it is not real hardware. -->
+   <xacro:cylinder_inertia  r="${wheel_radius}" l="${wheel_length}"  mass="5" />
    <visual>
     <origin rpy="0 0 1.5707" xyz="0 0 0"/>
@@ -144,6 +159,6 @@
 <!-- #######################################################################################################-->
 <link name="support_right_wheel_link">
-  <!-- Support roller, ~5 kg (0.4 m dia x 0.3 m rubber roller). -->
-  <xacro:cylinder_inertia r="0.2" l="${wheel_length}" mass="5"/>
+  <!-- Support roller: steel roller with rubber rim, ~20 kg. -->
+  <xacro:cylinder_inertia r="0.2" l="${wheel_length}" mass="20"/>
   <visual>
       <origin rpy="0 1.5707 1.5707" xyz="0 0 0"/>
@@ -169,6 +184,6 @@
 <!-- #######################################################################################################-->
 <link name="support_left_wheel_link">
-  <!-- Support roller, ~5 kg (0.4 m dia x 0.3 m rubber roller). -->
-  <xacro:cylinder_inertia r="0.2" l="${wheel_length}" mass="5"/>
+  <!-- Support roller: steel roller with rubber rim, ~20 kg. -->
+  <xacro:cylinder_inertia r="0.2" l="${wheel_length}" mass="20"/>
   <visual>
       <origin rpy="0 1.5707 1.5707" xyz="0 0 0"/>
@@ -214,9 +229,14 @@
   <!-- Belt collision: flat bottom box (like the official gz-sim tracked
        vehicle example) plus rounded ends. On a mesh terrain the flat box
-       gives many contact points; the cylinders roll over edges. -->
-  <collision>
-    <origin rpy="0 0 0" xyz="1.28 ${y_off} 0.09"/>
-    <geometry>
-      <box size="1.25 0.3 0.1"/>
+       gives many contact points; the cylinders roll over edges. The box
+       spans exactly the flat bottom run of the visible belt band mesh
+       (link x from the rear wheel tangent 0.555 to the front wheel
+       tangent 1.755), so the collision footprint matches the visible
+       track. The rear edge position matters for slope stability: the
+       machine is rated for ~60 deg climbs. -->
+  <collision>
+    <origin rpy="0 0 0" xyz="1.155 ${y_off} 0.09"/>
+    <geometry>
+      <box size="1.2 0.3 0.1"/>
     </geometry>
   </collision>
@@ -235,29 +255,36 @@
 </xacro:macro>
 <gazebo reference="track_left_wheel_link">
-  <!-- Rubber belt with steel grousers on soil. Rubber on dry soil is
-       ~0.6-0.8, but grousers mechanically engage the soil, giving a
-       coefficient of traction around 1.0-1.2 (tracked machines climb
-       ~40-50 deg slopes in reality). 1.2 holds the robot static on
-       slopes up to atan(1.2) ~ 50 deg, covering the forest terrains
-       (steepest sustained slopes: ~29 deg easy, ~37-47 deg medium).
+  <!-- Rubber belt with steel grousers on firm soil. Rubber on dry soil
+       is ~0.6-0.8; steel grousers interlock with the soil surface,
+       which on firm ground pushes the traction coefficient to ~2.0.
+       The REAL machine drives up ~60 deg slopes, which needs
+       mu > tan(60) = 1.73, so 2.0 gives it ~15% traction margin.
+       NOTE: the engine combines the two contacting surfaces
+       conservatively (effective ~ min of the pair), so the terrain
+       models in models/ground-*/model.sdf carry the same 2.0 —
+       leaving them at the SDF default 1.0 would cap the grip again.
        Isotropic on purpose: the grip must not depend on the engine
        honouring anisotropic friction, and skid steering still works
        (TrackedVehicle forces lateral slip via differential track
        speeds). -->
-  <mu1>1.2</mu1>
-  <mu2>1.2</mu2>
+  <mu1>2.0</mu1>
+  <mu2>2.0</mu2>
 </gazebo>
 <gazebo reference="track_right_wheel_link">
-  <mu1>1.2</mu1>
-  <mu2>1.2</mu2>
-</gazebo>
-<!-- Non-driving contact surfaces. The hull has ~21 cm ground clearance
-     and the belt is the lowest point, so these only touch on large
-     bumps or side slopes; they get realistic material friction
-     (steel hull/stabilizer/mulcher ~0.3 on soil, rubber rollers and
-     road wheels ~0.8) while the belt supplies the traction. Note the
-     URDF->SDF converter applies each block to the collisions of that
-     exact link only, so every fixed-jointed body part needs its own
-     block (they get lumped into chassis_link but keep their names). -->
+  <mu1>2.0</mu1>
+  <mu2>2.0</mu2>
+</gazebo>
+<!-- Contact surfaces besides the belt. The hull has ~21 cm ground
+     clearance and the belt is the lowest point, so these only touch on
+     large bumps or side slopes. The rollers, road wheels and the tail
+     stabilizer carry the SAME high grip as the belt (2.0): they are
+     part of the traction system, and a low-mu contact there was
+     measured to drag the robot down steep slopes (a 0.3 stabilizer
+     broke the static hold past ~51 deg). The bare hull and the
+     mulcher keep ~0.3 (steel sliding on soil / cutting drum). Note
+     the URDF->SDF converter applies each block to the collisions of
+     that exact link only, so every fixed-jointed body part needs its
+     own block (they get lumped into chassis_link but keep their
+     names). -->
 <gazebo reference="chassis_link">
   <mu1>0.3</mu1>
@@ -265,14 +292,14 @@
 </gazebo>
 <gazebo reference="stabilizer_link">
-  <mu1>0.3</mu1>
-  <mu2>0.3</mu2>
+  <mu1>2.0</mu1>
+  <mu2>2.0</mu2>
 </gazebo>
 <gazebo reference="support_left_wheel_link">
-  <mu1>0.8</mu1>
-  <mu2>0.8</mu2>
+  <mu1>2.0</mu1>
+  <mu2>2.0</mu2>
 </gazebo>
 <gazebo reference="support_right_wheel_link">
-  <mu1>0.8</mu1>
-  <mu2>0.8</mu2>
+  <mu1>2.0</mu1>
+  <mu2>2.0</mu2>
 </gazebo>
 <gazebo reference="tool_link">
@@ -280,13 +307,17 @@
   <mu2>0.3</mu2>
 </gazebo>
-<!-- Road wheels inside the belt: rubber, they sit ~9 mm above the
-     belt bottom and only touch on soft ground. -->
+<!-- Road wheels and support rollers inside the belt: they sit
+     ~1 cm above the belt bottom and only touch when terrain pushes
+     through the belt (bumps, soft ground). They are part of the
+     traction system: when they contact, they must grip like the
+     belt instead of dragging (a low-mu roller contact was found
+     to break the static hold on steep slopes). -->
 <gazebo reference="right_wheel_link">
-  <mu1>0.8</mu1>
-  <mu2>0.8</mu2>
+  <mu1>2.0</mu1>
+  <mu2>2.0</mu2>
 </gazebo>
 <gazebo reference="left_wheel_link">
-  <mu1>0.8</mu1>
-  <mu2>0.8</mu2>
+  <mu1>2.0</mu1>
+  <mu2>2.0</mu2>
 </gazebo>
 <!-- Tracked-vehicle conversion: the track links carry the belt        -->
@@ -305,8 +336,8 @@
            robot backwards onto its tail stabilizer). -->
       <origin xyz="1.38 0 0.3755"/>
-      <!-- 250 kg per side: rubber belt + steel grousers + rollers of a
+      <!-- 400 kg per side: rubber belt + steel grousers + rollers of a
            ~1.9 m track. Inertia of a 2.0 x 0.3 x 0.9 m box about its
            center. -->
-      <mass value="250"/>
+      <mass value="400"/>
       <inertia ixx="18.75" ixy="0" ixz="0" iyy="100.21" iyz="0" izz="85.21"/>
     </inertial>
@@ -328,8 +359,8 @@
            robot backwards onto its tail stabilizer). -->
       <origin xyz="1.38 0 0.3755"/>
-      <!-- 250 kg per side: rubber belt + steel grousers + rollers of a
+      <!-- 400 kg per side: rubber belt + steel grousers + rollers of a
            ~1.9 m track. Inertia of a 2.0 x 0.3 x 0.9 m box about its
            center. -->
-      <mass value="250"/>
+      <mass value="400"/>
       <inertia ixx="18.75" ixy="0" ixz="0" iyy="100.21" iyz="0" izz="85.21"/>
     </inertial>
